Commit message: Snapshot robot workspace before odometry fixes
Baseline of the current working state: EKF config, laser filter,
URDF camera link, Cartographer/Nav2 tuning, ArUco node and camera
calibration. No code changes.

Co-Authored-By: Claude Opus 5.5 <noreply@anthropic.com>

File: src/ired_bringup/urdf/ired.urdf.xacro (robot description, xacro)
@@ -23,5 +23,5 @@
         <parent link="base_link"/>
         <child link="aruco_camera_link"/>
-        <origin xyz="0.0 0.0 0.0" rpy="0.0 0.0 0.0"/>
+        <origin xyz="0.0 0.0 0.335" rpy="0.0 0.0 0.0"/>
     </joint>
     <joint name="base_cartesian_joint" type="fixed">

Commit message: A1: let the EKF use the IMU
imu.py stamps its data with frame imu_link, but the omni URDF had no
such link, so robot_localization dropped every IMU message and the
filtered odometry was wheel-only. Add imu_link (fixed to base_link,
same as the default main-branch URDF) and give the IMU realistic
covariances instead of all zeros.

Co-Authored-By: Claude Opus 5.5 <noreply@anthropic.com>

File: src/ired_bringup/urdf/ired.urdf.xacro (robot description, xacro)
@@ -10,4 +10,5 @@
     <link name="aruco_camera_link"/>
     <link name="base_cartesian_link"/>
+    <link name="imu_link"/>
     <joint name="base_joint" type="fixed">
         <parent link="base_footprint"/>
@@ -28,4 +29,9 @@
         <parent link="base_link"/>
         <child link="base_cartesian_link"/>
+        <origin xyz="0.0 0.0 0.0" rpy="0.0 0.0 0.0"/>
+    </joint>
+    <joint name="imu_joint" type="fixed">
+        <parent link="base_link"/>
+        <child link="imu_link"/>
         <origin xyz="0.0 0.0 0.0" rpy="0.0 0.0 0.0"/>
     </joint>

Commit message: Show the robot 3D model on base_link
Reduced Robocup_MobileRobot.stl from 1.06M to 100k faces (53 MB to
5 MB) so RViz and the web viewer stay fast on the Pi, and attached it
as a visual-only mesh on base_link. Links, joints and frames are
unchanged.

Co-Authored-By: Claude Opus 5.5 <noreply@anthropic.com>

File: src/ired_bringup/urdf/ired.urdf.xacro (robot description, xacro)
@@ -2,5 +2,17 @@
 <robot name="IRED">
     <link name="base_footprint"/>
-    <link name="base_link"/>
+    <link name="base_link">
+        <!-- 3D model for display only (no collision). The STL is in mm with its
+             floor at z=-30.6 mm and the base centre at (-94.0, 4.8) mm, so this
+             origin puts that centre on base_link (0.11 m above the floor).
+             If the model faces the wrong way, use rpy="0 0 3.14159" and
+             xyz="-0.094 0.005 -0.0794". -->
+        <visual>
+            <origin xyz="0.094 -0.005 -0.0794" rpy="0.0 0.0 0.0"/>
+            <geometry>
+                <mesh filename="package://ired_bringup/meshes/ired_body.stl" scale="0.001 0.001 0.001"/>
+            </geometry>
+        </visual>
+    </link>
     <link name="wheel_front_left_link"/>
     <link name="wheel_front_right_link"/>

Commit message: URDF: put the ArUco camera where it really is
The camera joint was at the robot centre, 0.445 m above the floor.
The camera hangs under the LiDAR plate, 0.23 m in front of the centre
(from the 3D model) and 0.29 m above the floor (measured), so marker
positions in base_link were off by about 0.23 m.

Co-Authored-By: Claude Opus 5.5 <noreply@anthropic.com>

File: src/ired_bringup/urdf/ired.urdf.xacro (robot description, xacro)
@@ -33,8 +33,11 @@
         <origin xyz="0.0 0.0 0.285" rpy="0.0 0.0 0.0"/>
     </joint>
+    <!-- Camera lens is 0.23 m in front of the centre (from the 3D model) and 0.29 m above
+         the floor (measured); base_link is 0.11 m above the floor.
+         Keep colons out of comments here, bringup.launch.py parses this file as YAML. -->
     <joint name="aruco_camera_joint" type="fixed">
         <parent link="base_link"/>
         <child link="aruco_camera_link"/>
-        <origin xyz="0.0 0.0 0.335" rpy="0.0 0.0 0.0"/>
+        <origin xyz="0.23 0.0 0.18" rpy="0.0 0.0 0.0"/>
     </joint>
     <joint name="base_cartesian_joint" type="fixed">

Commit message: URDF: turn the 3D model to face the robot front
The camera and arm are at -X in the STL but the robot drives along +X, so the model showed backwards. Rotate the visual 180 deg about Z (display only).

Co-Authored-By: Claude Opus 5.5 <noreply@anthropic.com>

File: src/ired_bringup/urdf/ired.urdf.xacro (robot description, xacro)
@@ -6,8 +6,7 @@
              floor at z=-30.6 mm and the base centre at (-94.0, 4.8) mm, so this
              origin puts that centre on base_link (0.11 m above the floor).
-             If the model faces the wrong way, use rpy="0 0 3.14159" and
-             xyz="-0.094 0.005 -0.0794". -->
+             The robot front (camera and arm) is -X in the STL, hence the 180 deg yaw. -->
         <visual>
-            <origin xyz="0.094 -0.005 -0.0794" rpy="0.0 0.0 0.0"/>
+            <origin xyz="-0.094 0.005 -0.0794" rpy="0.0 0.0 3.14159"/>
             <geometry>
                 <mesh filename="package://ired_bringup/meshes/ired_body.stl" scale="0.001 0.001 0.001"/>

Commit message: PROPOSAL URDF: camera low at the front, LiDAR at 0.32 m (new model)
From Robocup_MobileRobot.stl / .step of 2026-10-19:
- aruco_camera_joint 0.23 0 0.18 -> 0.25 0 0.023: C270 front face 0.26 m
  ahead of the centre, lens ~0.25 m, centre 0.133 m above the floor (was
  0.29 m), close to the ArUco centre on the boxes (~0.10 m).
- scan_joint 0.285 -> 0.21 above base_link: RPLidar A1 head on the robot
  centre at 0.31-0.33 m, laser plane ~0.32 m above the floor. Yaw kept.
- visual origin for the new body STL (base centre -91.3, 1.9 mm in the STL).
The camera position needs a new camera calibration once mounted.

Co-Authored-By: Claude Opus 5.5 <noreply@anthropic.com>

File: src/ired_bringup/urdf/ired.urdf.xacro (robot description, xacro)
@@ -3,10 +3,11 @@
     <link name="base_footprint"/>
     <link name="base_link">
-        <!-- 3D model for display only (no collision). The STL is in mm with its
-             floor at z=-30.6 mm and the base centre at (-94.0, 4.8) mm, so this
-             origin puts that centre on base_link (0.11 m above the floor).
-             The robot front (camera and arm) is -X in the STL, hence the 180 deg yaw. -->
+        <!-- 3D model for display only (no collision), from Robocup_MobileRobot.stl of
+             2026-10-19 reduced to about 110k triangles. The STL is in mm with its floor
+             at z=-30.6 mm and the base centre at (-91.3, 1.9) mm, so this origin puts
+             that centre on base_link (0.11 m above the floor). The robot front (camera)
+             is -X in the STL, hence the 180 deg yaw. The SCARA arm is drawn unfolded. -->
         <visual>
-            <origin xyz="-0.094 0.005 -0.0794" rpy="0.0 0.0 3.14159"/>
+            <origin xyz="-0.0913 0.0019 -0.0794" rpy="0.0 0.0 3.14159"/>
             <geometry>
                 <mesh filename="package://ired_bringup/meshes/ired_body.stl" scale="0.001 0.001 0.001"/>
@@ -27,16 +28,20 @@
         <origin xyz="0.0 0.0 0.11" rpy="0.0 0.0 0.0"/>
     </joint>
+    <!-- RPLidar A1 head on the robot centre, laser plane about 0.32 m above the floor
+         (head 0.31 to 0.33 m in the 2026-10-19 model), so 0.21 m above base_link.
+         Yaw unchanged, the scan orientation was already checked against odometry. -->
     <joint name="scan_joint" type="fixed">
         <parent link="base_link"/>
         <child link="base_scan"/>
-        <origin xyz="0.0 0.0 0.285" rpy="0.0 0.0 0.0"/>
+        <origin xyz="0.0 0.0 0.21" rpy="0.0 0.0 0.0"/>
     </joint>
-    <!-- Camera lens is 0.23 m in front of the centre (from the 3D model) and 0.29 m above
-         the floor (measured); base_link is 0.11 m above the floor.
+    <!-- C270 camera, level, lens about 0.25 m in front of the centre (front face 0.26 m)
+         and 0.133 m above the floor (2026-10-19 model), base_link is 0.11 m above the
+         floor. Low enough to see the ArUco markers (centre about 0.10 m) straight on.
          Keep colons out of comments here, bringup.launch.py parses this file as YAML. -->
     <joint name="aruco_camera_joint" type="fixed">
         <parent link="base_link"/>
         <child link="aruco_camera_link"/>
-        <origin xyz="0.23 0.0 0.18" rpy="0.0 0.0 0.0"/>
+        <origin xyz="0.25 0.0 0.023" rpy="0.0 0.0 0.0"/>
     </joint>
     <joint name="base_cartesian_joint" type="fixed">

Commit message: ired_bringup: URDF for the updated robot model (2026-10-19 evening)
New Robocup_MobileRobot.stl: floor at z=65.7 mm in the STL (visual origin
z -0.0794 -> -0.1757), laser plane about 0.295 m above the floor (scan_joint
z 0.21 -> 0.185), camera centre about 0.12 m (aruco_camera_joint z 0.023 ->
0.010). Wheel centre, camera reach (0.26 m) and the four posts are unchanged.
LiDAR yaw stays 0: the CAD draws it turned 180 deg, on the robot its motor
side points forward. Mesh reduced to 112k triangles as before.

Co-Authored-By: Claude Opus 5.5 <noreply@anthropic.com>

File: src/ired_bringup/urdf/ired.urdf.xacro (robot description, xacro)
@@ -4,10 +4,12 @@
     <link name="base_link">
         <!-- 3D model for display only (no collision), from Robocup_MobileRobot.stl of
-             2026-10-19 reduced to about 110k triangles. The STL is in mm with its floor
-             at z=-30.6 mm and the base centre at (-91.3, 1.9) mm, so this origin puts
-             that centre on base_link (0.11 m above the floor). The robot front (camera)
-             is -X in the STL, hence the 180 deg yaw. The SCARA arm is drawn unfolded. -->
+             2026-10-19 evening (updated frame) reduced to about 110k triangles. The STL is in mm
+             with its floor at z=65.7 mm and the wheel centre at (-91.3, 1.9) mm as before,
+             so this origin puts that centre on base_link (0.11 m above the floor). The robot
+             front (camera) is -X in the STL, hence the 180 deg yaw. The SCARA arm is drawn
+             unfolded, and the RPLidar is drawn turned 180 deg (CAD only, on the robot its
+             motor side points forward). -->
         <visual>
-            <origin xyz="-0.0913 0.0019 -0.0794" rpy="0.0 0.0 3.14159"/>
+            <origin xyz="-0.0913 0.0019 -0.1757" rpy="0.0 0.0 3.14159"/>
             <geometry>
                 <mesh filename="package://ired_bringup/meshes/ired_body.stl" scale="0.001 0.001 0.001"/>
@@ -28,20 +30,21 @@
         <origin xyz="0.0 0.0 0.11" rpy="0.0 0.0 0.0"/>
     </joint>
-    <!-- RPLidar A1 head on the robot centre, laser plane about 0.32 m above the floor
-         (head 0.31 to 0.33 m in the 2026-10-19 model), so 0.21 m above base_link.
-         Yaw unchanged, the scan orientation was already checked against odometry. -->
+    <!-- RPLidar A1 head on the robot centre, laser plane about 0.295 m above the floor
+         (head top 0.30 m in the updated model, 26 mm lower than before), so 0.185 m above
+         base_link. Measure the real plane on the robot. Yaw unchanged, the scan orientation
+         was already checked against odometry and the motor side points forward. -->
     <joint name="scan_joint" type="fixed">
         <parent link="base_link"/>
         <child link="base_scan"/>
-        <origin xyz="0.0 0.0 0.21" rpy="0.0 0.0 0.0"/>
+        <origin xyz="0.0 0.0 0.185" rpy="0.0 0.0 0.0"/>
     </joint>
     <!-- C270 camera, level, lens about 0.25 m in front of the centre (front face 0.26 m)
-         and 0.133 m above the floor (2026-10-19 model), base_link is 0.11 m above the
-         floor. Low enough to see the ArUco markers (centre about 0.10 m) straight on.
+         and 0.12 m above the floor (camera block 0.101 to 0.138 m in the updated model),
+         base_link is 0.11 m above the floor. Low enough to see the ArUco markers (centre about 0.10 m) straight on.
          Keep colons out of comments here, bringup.launch.py parses this file as YAML. -->
     <joint name="aruco_camera_joint" type="fixed">
         <parent link="base_link"/>
         <child link="aruco_camera_link"/>
-        <origin xyz="0.25 0.0 0.023" rpy="0.0 0.0 0.0"/>
+        <origin xyz="0.25 0.0 0.010" rpy="0.0 0.0 0.0"/>
     </joint>
     <joint name="base_cartesian_joint" type="fixed">
